File: OnonoKey1.kicad_pcb (KiCad board)
At the start: 2 copper layers, 136.9 x 136.4 mm, 97 parts, among them SW00 Switch, SW01 Switch, SW02 Switch, SW03 Switch, SW04 Switch, SW05 Switch, SW06 Switch, SW10 Switch, SW11 Switch, SW12 Switch, SW13 Switch, SW14 Switch, SW15 Switch, SW16 Switch, SW20 Switch, SW21 Switch, SW22 Switch, SW23 Switch, SW24 Switch, SW25 Switch, SW26 Switch, SW30 Switch, SW31 Switch, SW32 Switch, SW33 Switch, SW34 Switch, SW35 Switch, SW36 Switch, SW40 Switch, SW41 Switch, SW42 Switch, SW43 Switch, SW44 Switch, SW45 Switch, SW46 Switch, SW50 Switch, SW51 Switch, SW52 Switch, SW53 Switch, SW54 Switch, SW55 Switch, SW56 Switch, U1 RP2040_Zero, U2 TRRS Front, U3 TRRS Back

Commit message: Included used footprints and links to sources, hopefully pcb file works out of the box
Parts:
- D1, D10, D11, D12, D13, D14, D15, D16, D17, D18, D19, D2, D20, D21, D22, D23, D24, D25, D26, D27, D28, D29, D3, D30, D31, D32, D33, D34, D35, D36, D37, D38, D39, D4, D40, D41, D42, D5, D6, D7, D8, D9: footprint ScottoKeebs_Components:Diode_DO-35 -> used-footprints:Diode_DO-35
- REF** (x8): footprint MountingHole:MountingHole_2.2mm_M2 -> used-footprints:MountingHole_2.2mm_M2
- REF** (x2): footprint MountingHole:MountingHole_2.7mm_M2.5_DIN965 -> used-footprints:MountingHole_2.7mm_M2.5_DIN965
- SW00, SW01, SW02, SW03, SW04, SW05, SW06, SW10, SW11, SW12, SW13, SW14, SW15, SW16, SW20, SW21, SW22, SW23, SW24, SW25, SW26, SW30, SW31, SW32, SW33, SW34, SW35, SW36, SW40, SW41, SW42, SW43, SW44, SW45, SW46, SW50, SW51, SW52, SW53, SW54, SW55, SW56: footprint Daprice_Keyswitches:Kailh_socket_MX_optional_reversible_1u -> used-footprints:Kailh_socket_MX_optional_reversible_1u
- U1: footprint ScottoKeebs_MCU:RP2040_Zero -> used-footprints:RP2040_Zero
- U2, U3: footprint ScottoKeebs_Components:TRRS_PJ-320A -> used-footprints:TRRS_PJ-320A
